File: hw/left/keeb-left.kicad_pcb (KiCad board)
At the start: 2 copper layers, 105.8 x 97 mm, 45 parts, among them J1 USB4105-GF-A, J2 SJ2-3574A-SMT-TR, J3 Conn_01x04_Pin, U1 ATmega32U2-A, U2 PTS526 SK15 SMTR2 LFS, Y1 16MHz

Commit message: Hardware revision
Other:
- board text added: "JLCJLCJLCJLC"
Changed lines of the file:
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@@
 		(tags "PTS526 SK15 SMTR2 LFS ")
 		(property "Reference" "U2"
-			(at 0 0 180)
+			(at 0 0 0)
 			(unlocked yes)
 			(layer "F.SilkS")
@@
 		(fp_text user "*"
 			(at -3.43535 -3.556 180)
+			(unlocked yes)
 			(layer "F.SilkS")
 			(effects
@@
 		(fp_text user "*"
 			(at -3.43535 -3.556 180)
-			(unlocked yes)
 			(layer "F.SilkS")
 			(effects
@@
 		(fp_text user "*"
 			(at -2.3241 -2.6289 180)
+			(unlocked yes)
 			(layer "F.Fab")
 			(effects
@@
 		(fp_text user "*"
 			(at -2.3241 -2.6289 180)
-			(unlocked yes)
 			(layer "F.Fab")
 			(effects
@@
 		(layer "Edge.Cuts")
 	)
+	(gr_text "JLCJLCJLCJLC"
+		(at 116.90572 137.308554 0)
+		(layer "B.SilkS")
+		(effects
+			(font
+				(size 1 1)
+				(thickness 0.1)
+			)
+			(justify left bottom mirror)
+		)
+	)
 	(gr_text "MOSI"
