File: hw/right/keeb-right.kicad_pcb (KiCad board)
At the start: 2 copper layers, 105.8 x 97 mm, 45 parts, among them J1 USB4105-GF-A, J2 SJ2-3574A-SMT-TR, J3 Conn_01x04_Pin, U1 ATmega32U2-A, U2 PTS526 SK15 SMTR2 LFS, Y1 16MHz

Commit message: Hardware revision
Parts:
- added C2: 20pf, Capacitor_SMD:C_0805_2012Metric, F.Cu at (98.1, 136.3)
- added C3: 20pf, Capacitor_SMD:C_0805_2012Metric, F.Cu at (99.6, 134.8)
Connections:
- J2 pad 2: TX -> RX
- J2 pad 3: RX -> TX
Routing:
- net TX: track 63.4 -> 69.9 mm
- net Net-(U1-PC0/XTAL2): track 34.4 -> 39.2 mm
- net GND: track 104.6 -> 109.1 mm
- net Net-(U1-XTAL1): track 21.1 -> 24.1 mm
- net RX: track 59.9 -> 61.1 mm
Other:
- board text added: "JLCJLCJLCJLC"
