File: hw/right/keeb-right.kicad_sch (KiCad schematic)
At the start: 42 parts, among them J1 USB4105-GF-A, J2 SJ2-3574A-SMT-TR, J3 Conn_01x04_Pin, U1 ATmega32U2-A, U2 PTS526 SK15 SMTR2 LFS, Y1 16MHz

Commit message: Hardware revision
Connections:
- net RX: now also J2.2; no longer J2.3
- net TX: now also J2.3; no longer J2.2

Commit message: Update hardware
Parts:
- R10, R7, R8, R9: value 220 -> 10k
Other:
- note added: "1.1"
- note added: "5/14/25"
- note added: "Keeb"
- note removed: "1"
- note removed: "4/17/25"
- note removed: "Ergo-keyboard"
Changed lines of the file:
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@@
 		)
 	)
-	(text "1"
+	(text "1.1"
 		(exclude_from_sim no)
 		(at 275.082 193.294 0)
@@
 		)
 	)
-	(text "Ergo-keyboard"
+	(text "Keeb"
 		(exclude_from_sim no)
-		(at 195.326 189.738 0)
+		(at 188.976 189.738 0)
 		(effects
 			(font
@@
 		)
 	)
-	(text "4/17/25"
+	(text "5/14/25"
 		(exclude_from_sim no)
 		(at 212.344 193.294 0)
@@
 			)
 		)
-		(property "Value" "220"
+		(property "Value" "10k"
 			(at 100.33 163.8299 0)
 			(effects
@@
 			)
 		)
-		(property "Value" "220"
+		(property "Value" "10k"
 			(at 166.37 92.71 90)
 			(effects
@@
 			)
 		)
-		(property "Value" "220"
+		(property "Value" "10k"
 			(at 176.53 125.7299 0)
 			(effects
@@
 			)
 		)
-		(property "Value" "220"
+		(property "Value" "10k"
 			(at 187.96 125.7299 0)
 			(effects
